File: _Start Here - New PCB/StartHere.brd (EAGLE design)
At the start: 100 x 75 mm, 1 part

Commit message: Still Syncing to GIT
Still Syncing to GIT
Parts:
- removed C7: 47u, capacitor-wima:C7.5B3
Connections:
- removed net N$4: C7.1
- removed net V+: C7.2
Routing:
- net N$39: track 7.19 -> 0.00 mm
- net N$29: track 1.27 -> 0.00 mm
- removed copper zone on layer 16, net GND
Changed lines of the file:
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@@
 <layer number="43" name="vRestrict" color="2" fill="10" visible="yes" active="yes"/>
 <layer number="44" name="Drills" color="7" fill="1" visible="no" active="yes"/>
-<layer number="45" name="Holes" color="7" fill="1" visible="yes" active="yes"/>
+<layer number="45" name="Holes" color="7" fill="1" visible="no" active="yes"/>
 <layer number="46" name="Milling" color="3" fill="1" visible="no" active="yes"/>
 <layer number="47" name="Measures" color="7" fill="1" visible="no" active="yes"/>
@@
 <layer number="97" name="Info" color="7" fill="1" visible="no" active="no"/>
 <layer number="98" name="Guide" color="6" fill="1" visible="no" active="no"/>
-<layer number="99" name="SpiceOrder" color="5" fill="1" visible="no" active="no"/>
 </layers>
 <board>
@@
 <wire x1="100" y1="75" x2="0" y2="75" width="0" layer="20"/>
 <wire x1="0" y1="75" x2="0" y2="0" width="0" layer="20"/>
-<circle x="26.67" y="15.24" radius="0.85" width="1" layer="16"/>
-<circle x="6.5" y="68.5" radius="1.8" width="0.25" layer="19"/>
-<circle x="6.5" y="6.5" radius="1.8" width="0.25" layer="19"/>
-<circle x="93.5" y="6.5" radius="1.8" width="0.25" layer="19"/>
-<circle x="93.5" y="68.5" radius="1.8" width="0.25" layer="19"/>
+<circle x="6.5" y="68.5" radius="1.8" width="0.254" layer="19"/>
+<circle x="93.5" y="68.5" radius="1.8" width="0.254" layer="19"/>
+<circle x="93.5" y="6.5" radius="1.8" width="0.254" layer="19"/>
+<circle x="6.5" y="6.5" radius="1.8" width="0.254" layer="19"/>
 </plain>
 <attributes>
@@
 <param name="TopRouterVariant" value="1"/>
 <param name="tpViaShape" value="round"/>
-<param name="PrefDir.1" value="0"/>
+<param name="PrefDir.1" value="a"/>
 <param name="PrefDir.2" value="0"/>
 <param name="PrefDir.3" value="0"/>
@@
 </autorouter>
 <elements>
-<element name="C7" library="capacitor-wima" package="C7.5B3" value="47u" x="61.595" y="7.62" rot="R90"/>
 </elements>
 <signals>
-<signal name="GND">
-<polygon width="0.254" layer="16" spacing="0.4064">
-<vertex x="0" y="0"/>
-<vertex x="0" y="75"/>
-<vertex x="100" y="75"/>
-<vertex x="100" y="0"/>
-</polygon>
-</signal>
-<signal name="V+">
-<contactref element="C7" pad="2"/>
-<wire x1="79.375" y1="31.75" x2="75.565" y2="58.42" width="0" layer="19" extent="1-1"/>
-<wire x1="61.595" y1="11.43" x2="79.375" y2="31.75" width="0" layer="19" extent="1-1"/>
-</signal>
-<signal name="N$20">
-</signal>
-<signal name="N$23">
-</signal>
-<signal name="N$24">
-</signal>
-<signal name="N$25">
-</signal>
-<signal name="N$26">
-</signal>
-<signal name="N$27">
-</signal>
-<signal name="N$28">
-</signal>
-<signal name="N$29">
-<wire x1="31.75" y1="12.7" x2="33.02" y2="12.7" width="2.1844" layer="16"/>
-</signal>
-<signal name="N$34">
-</signal>
-<signal name="N$31">
-</signal>
-<signal name="N$30">
-</signal>
-<signal name="N$32">
-</signal>
-<signal name="N$35">
-</signal>
-<signal name="N$36">
-</signal>
-<signal name="N$37">
-</signal>
-<signal name="N$38">
-</signal>
-<signal name="N$39">
-<wire x1="5.715" y1="47.625" x2="6.35" y2="49.53" width="1.016" layer="16"/>
-<wire x1="6.35" y1="49.53" x2="5.715" y2="49.53" width="1.016" layer="16"/>
-<wire x1="5.715" y1="49.53" x2="5.08" y2="49.53" width="1.016" layer="16"/>
-<wire x1="5.08" y1="49.53" x2="5.715" y2="47.625" width="1.016" layer="16"/>
-<wire x1="5.715" y1="47.625" x2="5.715" y2="49.53" width="1.016" layer="16"/>
-</signal>
-<signal name="N$4">
-<contactref element="C7" pad="1"/>
-<wire x1="71.755" y1="16.51" x2="67.945" y2="43.18" width="0" layer="19" extent="1-1"/>
-<wire x1="61.595" y1="3.81" x2="71.755" y2="16.51" width="0" layer="19" extent="1-1"/>
-</signal>
 </signals>
 </board>
